File: hardware/edf-esc.kicad_sch (KiCad schematic)
At the start: 0 parts

Commit message: feat: add connected dual ESC schematic
Parts:
- added QA1, QA10, QA11, QA12, QA13, QA14, QA15, QA16, QA17, QA18, QA2, QA3, QA4, QA5, QA6, QA7, QA8, QA9, QB1, QB10, QB11, QB12, QB13, QB14, QB15, QB16, QB17, QB18, QB2, QB3, QB4, QB5, QB6, QB7, QB8, QB9: SFS06R025GF, symbol EDF_ESC:SFS06R025GF
- added RGA1, RGA10, RGA11, RGA12, RGA13, RGA14, RGA15, RGA16, RGA17, RGA18, RGA2, RGA3, RGA4, RGA5, RGA6, RGA7, RGA8, RGA9, RGB1, RGB10, RGB11, RGB12, RGB13, RGB14, RGB15, RGB16, RGB17, RGB18, RGB2, RGB3, RGB4, RGB5, RGB6, RGB7, RGB8, RGB9: 4R7, symbol EDF_ESC:R_0603
- added U12V: XL1509-ADJ, symbol EDF_ESC:XL1509-ADJ
- added U3V3: XC6206P332MR, symbol EDF_ESC:XC6206P332MR
- added UBEC: XL4016E1, symbol EDF_ESC:XL4016E1
- added UCA, UCB: PY32F030K28U6TR, symbol EDF_ESC:PY32F030K28U6TR
- added UCSA, UCSB: INA190A3IDDFR, symbol EDF_ESC:INA190A3IDDFR
- added UGA, UGB: DRV8300DRGER, symbol EDF_ESC:DRV8300DRGER
Other:
- note added: "UNVALIDATED — REVIEW ONLY; DO NOT FABRICATE"
- note removed: "AUXILIARY: XL1509-ADJ 12V GATE; XL4016E1 5V/8A TARGET; XC6206P332MR 3V3"
- note removed: "BEMF_A_U BEMF_A_V BEMF_A_W TIM1_BKIN_A"
- note removed: "BEMF_B_U BEMF_B_V BEMF_B_W TIM1_BKIN_B"
- note removed: "ESC A: DRV8300DRGER + 18x PARALLEL MOSFET + PY32F030K28U6TR"
- note removed: "ESC B: DRV8300DRGER + 18x PARALLEL MOSFET + PY32F030K28U6TR"
- note removed: "FET MANIFEST: SFS06R025GF SFS06R025GF SFS06R025GF SFS06R025GF SFS06R025GF SFS06R025GF SFS06R025GF SFS06R025GF SFS06R025GF SFS06R025GF SFS06R025GF SFS06R025GF SFS06R025GF SFS06R025GF SFS06R025GF SFS06R025GF SFS06R025GF SFS06R025GF SFS06R025GF SFS06R025GF SFS06R025GF SFS06R025GF SFS06R025GF SFS06R025GF SFS06R025GF SFS06R025GF SFS06R025GF SFS06R025GF SFS06R025GF SFS06R025GF SFS06R025GF SFS06R025GF S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"
- note removed: "POWER INPUT A: BAT_A+ -> KELVIN_A+ / KELVIN_A- -> INA190A3IDDFR"
- note removed: "POWER INPUT B: BAT_B+ -> KELVIN_B+ / KELVIN_B- -> INA190A3IDDFR"
- note removed: "UNVALIDATED REVIEW SCHEMATIC — see docs/requirements-traceability.md"
